File: E12.kicad_pcb (KiCad board)
At the start: 4 copper layers, 18 x 6.2 mm, 21 parts, among them J3 59453-061110EDHLF, U1 WS2811, U2 WS2811, U3 WS2811, U4 WS2811

Commit message: mod: optimized for PCB assembly
Parts:
- J3: value 59453-061110EDHLF -> FFC
- R11, R12: value R -> n.f.
- RN1, RN2, RN3, RN4: value R_Pack04 -> 220
Other:
- rule pad_to_mask_clearance: 0.051 -> 0
Changed lines of the file:
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@@
     (pad_size 0.52 1)
     (pad_drill 0)
-    (pad_to_mask_clearance 0.051)
-    (solder_mask_min_width 0.1)
+    (pad_to_mask_clearance 0)
     (aux_axis_origin 0 0)
     (visible_elements 7FFFFFFF)
@@
       (effects (font (size 1 1) (thickness 0.15)))
     )
-    (fp_text value 59453-061110EDHLF (at 0.0508 3.6322 90) (layer F.Fab)
+    (fp_text value FFC (at 0.0508 3.6322 90) (layer F.Fab)
       (effects (font (size 1 1) (thickness 0.15)))
     )
+    (fp_line (start -2.25 1.75) (end -2.25 -1.45) (layer F.Fab) (width 0.127))
+    (fp_line (start -2.25 -1.45) (end -2.25 -1.75) (layer F.Fab) (width 0.127))
+    (fp_line (start 2.25 -1.75) (end 2.25 -1.45) (layer F.Fab) (width 0.127))
+    (fp_line (start 2.25 -1.45) (end 2.25 1.75) (layer F.Fab) (width 0.127))
+    (fp_line (start 2.25 1.75) (end -2.25 1.75) (layer F.Fab) (width 0.127))
+    (fp_line (start -2.25 -1.75) (end 2.25 -1.75) (layer F.Fab) (width 0.127))
+    (fp_line (start -2.25 -1.22) (end -2.25 -1.45) (layer F.SilkS) (width 0.127))
+    (fp_line (start -2.25 1.75) (end -2.25 0.42) (layer F.SilkS) (width 0.127))
+    (fp_line (start 2.25 -1.45) (end 2.25 -1.22) (layer F.SilkS) (width 0.127))
+    (fp_line (start 2.25 1.75) (end 2.25 0.42) (layer F.SilkS) (width 0.127))
+    (fp_line (start -2.25 -1.45) (end -1.72 -1.45) (layer F.SilkS) (width 0.127))
+    (fp_line (start 1.72 -1.45) (end 2.25 -1.45) (layer F.SilkS) (width 0.127))
+    (fp_line (start 2.25 1.75) (end -2.25 1.75) (layer F.SilkS) (width 0.127))
+    (fp_line (start -2.5 -2.8) (end -2.5 2) (layer F.CrtYd) (width 0.05))
+    (fp_line (start -2.5 2) (end 2.5 2) (layer F.CrtYd) (width 0.05))
+    (fp_line (start 2.5 2) (end 2.5 -2.8) (layer F.CrtYd) (width 0.05))
+    (fp_circle (center -1.25 -3.15) (end -1.15 -3.15) (layer F.SilkS) (width 0.2))
+    (fp_circle (center -1.25 -3.15) (end -1.15 -3.15) (layer F.Fab) (width 0.2))
+    (fp_line (start -2.25 -1.45) (end 2.25 -1.45) (layer F.Fab) (width 0.127))
+    (fp_line (start 2.5 -2.8) (end -2.5 -2.8) (layer F.CrtYd) (width 0.05))
+    (fp_poly (pts (xy -1.45 -2.6) (xy -1.05 -2.6) (xy -1.05 -1.1) (xy -1.45 -1.1)) (layer F.Mask) (width 0.01))
+    (fp_poly (pts (xy -0.95 -2.6) (xy -0.55 -2.6) (xy -0.55 -1.1) (xy -0.95 -1.1)) (layer F.Mask) (width 0.01))
+    (fp_poly (pts (xy -0.45 -2.6) (xy -0.05 -2.6) (xy -0.05 -1.1) (xy -0.45 -1.1)) (layer F.Mask) (width 0.01))
+    (fp_poly (pts (xy 0.05 -2.6) (xy 0.45 -2.6) (xy 0.45 -1.1) (xy 0.05 -1.1)) (layer F.Mask) (width 0.01))
+    (fp_poly (pts (xy 0.55 -2.6) (xy 0.95 -2.6) (xy 0.95 -1.1) (xy 0.55 -1.1)) (layer F.Mask) (width 0.01))
     (fp_poly (pts (xy 1.05 -2.6) (xy 1.45 -2.6) (xy 1.45 -1.1) (xy 1.05 -1.1)) (layer F.Mask) (width 0.01))
-    (fp_poly (pts (xy 0.55 -2.6) (xy 0.95 -2.6) (xy 0.95 -1.1) (xy 0.55 -1.1)) (layer F.Mask) (width 0.01))
-    (fp_poly (pts (xy 0.05 -2.6) (xy 0.45 -2.6) (xy 0.45 -1.1) (xy 0.05 -1.1)) (layer F.Mask) (width 0.01))
-    (fp_poly (pts (xy -0.45 -2.6) (xy -0.05 -2.6) (xy -0.05 -1.1) (xy -0.45 -1.1)) (layer F.Mask) (width 0.01))
-    (fp_poly (pts (xy -0.95 -2.6) (xy -0.55 -2.6) (xy -0.55 -1.1) (xy -0.95 -1.1)) (layer F.Mask) (width 0.01))
-    (fp_poly (pts (xy -1.45 -2.6) (xy -1.05 -2.6) (xy -1.05 -1.1) (xy -1.45 -1.1)) (layer F.Mask) (width 0.01))
-    (fp_line (start 2.5 -2.8) (end -2.5 -2.8) (layer F.CrtYd) (width 0.05))
-    (fp_line (start -2.25 -1.45) (end 2.25 -1.45) (layer F.Fab) (width 0.127))
-    (fp_circle (center -1.25 -3.15) (end -1.15 -3.15) (layer F.Fab) (width 0.2))
-    (fp_circle (center -1.25 -3.15) (end -1.15 -3.15) (layer F.SilkS) (width 0.2))
-    (fp_line (start 2.5 2) (end 2.5 -2.8) (layer F.CrtYd) (width 0.05))
-    (fp_line (start -2.5 2) (end 2.5 2) (layer F.CrtYd) (width 0.05))
-    (fp_line (start -2.5 -2.8) (end -2.5 2) (layer F.CrtYd) (width 0.05))
-    (fp_line (start 2.25 1.75) (end -2.25 1.75) (layer F.SilkS) (width 0.127))
-    (fp_line (start 1.72 -1.45) (end 2.25 -1.45) (layer F.SilkS) (width 0.127))
-    (fp_line (start -2.25 -1.45) (end -1.72 -1.45) (layer F.SilkS) (width 0.127))
-    (fp_line (start 2.25 1.75) (end 2.25 0.42) (layer F.SilkS) (width 0.127))
-    (fp_line (start 2.25 -1.45) (end 2.25 -1.22) (layer F.SilkS) (width 0.127))
-    (fp_line (start -2.25 1.75) (end -2.25 0.42) (layer F.SilkS) (width 0.127))
-    (fp_line (start -2.25 -1.22) (end -2.25 -1.45) (layer F.SilkS) (width 0.127))
-    (fp_line (start -2.25 -1.75) (end 2.25 -1.75) (layer F.Fab) (width 0.127))
-    (fp_line (start 2.25 1.75) (end -2.25 1.75) (layer F.Fab) (width 0.127))
-    (fp_line (start 2.25 -1.45) (end 2.25 1.75) (layer F.Fab) (width 0.127))
-    (fp_line (start 2.25 -1.75) (end 2.25 -1.45) (layer F.Fab) (width 0.127))
-    (fp_line (start -2.25 -1.45) (end -2.25 -1.75) (layer F.Fab) (width 0.127))
-    (fp_line (start -2.25 1.75) (end -2.25 -1.45) (layer F.Fab) (width 0.127))
     (pad 6 smd rect (at 1.25 -1.85 270) (size 0.3 1.4) (layers F.Cu F.Paste)
       (net 2 DI))
@@
       (net 4 VDD))
     (pad 8 smd rect (at 1.99 -0.4 270) (size 0.52 1) (layers F.Cu F.Paste F.Mask)
-      (net 1 GND) (solder_mask_margin 0.102) (zone_connect 2))
+      (net 1 GND) (solder_mask_margin 0.102) (zone_connect 1))
     (pad 7 smd rect (at -1.99 -0.4 270) (size 0.52 1) (layers F.Cu F.Paste F.Mask)
-      (net 1 GND) (solder_mask_margin 0.102) (zone_connect 2))
+      (net 1 GND) (solder_mask_margin 0.102))
     (pad 4 smd rect (at 0.25 -1.85 270) (size 0.3 1.4) (layers F.Cu F.Paste))
     (pad 3 smd rect (at -0.25 -1.85 270) (size 0.3 1.4) (layers F.Cu F.Paste))
@@
       (effects (font (size 1 1) (thickness 0.15)) (justify mirror))
     )
-    (fp_text value R (at 0 -1.65) (layer B.Fab)
+    (fp_text value n.f. (at 0 -1.65) (layer B.Fab)
       (effects (font (size 1 1) (thickness 0.15)) (justify mirror))
     )
@@
       (effects (font (size 0.5 0.5) (thickness 0.08)) (justify mirror))
     )
-    (pad 2 smd roundrect (at 0.9125 0 180) (size 1.025 1.4) (layers B.Cu B.Paste B.Mask) (roundrect_rratio 0.243902)
+    (pad 2 smd roundrect (at 0.9125 0 180) (size 1.025 1.4) (layers B.Cu B.Paste B.Mask) (roundrect_rratio 0.2439014634146341)
       (net 4 VDD))
-    (pad 1 smd roundrect (at -0.9125 0 180) (size 1.025 1.4) (layers B.Cu B.Paste B.Mask) (roundrect_rratio 0.243902)
+    (pad 1 smd roundrect (at -0.9125 0 180) (size 1.025 1.4) (layers B.Cu B.Paste B.Mask) (roundrect_rratio 0.2439014634146341)
       (net 2 DI))
     (model ${KISYS3DMOD}/Resistor_SMD.3dshapes/R_0805_2012Metric.wrl_
@@
       (effects (font (size 1 1) (thickness 0.15)) (justify mirror))
     )
-    (fp_text value R (at 0 -1.65) (layer B.Fab)
+    (fp_text value n.f. (at 0 -1.65) (layer B.Fab)
       (effects (font (size 1 1) (thickness 0.15)) (justify mirror))
     )
@@
       (effects (font (size 0.5 0.5) (thickness 0.08)) (justify mirror))
     )
-    (pad 2 smd roundrect (at 0.9125 0 180) (size 1.025 1.4) (layers B.Cu B.Paste B.Mask) (roundrect_rratio 0.243902)
+    (pad 2 smd roundrect (at 0.9125 0 180) (size 1.025 1.4) (layers B.Cu B.Paste B.Mask) (roundrect_rratio 0.2439014634146341)
       (net 1 GND))
-    (pad 1 smd roundrect (at -0.9125 0 180) (size 1.025 1.4) (layers B.Cu B.Paste B.Mask) (roundrect_rratio 0.243902)
+    (pad 1 smd roundrect (at -0.9125 0 180) (size 1.025 1.4) (layers B.Cu B.Paste B.Mask) (roundrect_rratio 0.2439014634146341)
       (net 3 DO))
     (model ${KISYS3DMOD}/Resistor_SMD.3dshapes/R_0805_2012Metric.wrl_
@@
       (effects (font (size 1 1) (thickness 0.15)) (justify mirror))
     )
-    (fp_text value R_Pack04 (at 0 -2.1) (layer B.Fab)
+    (fp_text value 220 (at 0 -2.1) (layer B.Fab)
       (effects (font (size 1 1) (thickness 0.15)) (justify mirror))
     )
@@
       (effects (font (size 1 1) (thickness 0.15)) (justify mirror))
     )
-    (fp_text value R_Pack04 (at 0 -2.1) (layer B.Fab)
+    (fp_text value 220 (at 0 -2.1) (layer B.Fab)
       (effects (font (size 1 1) (thickness 0.15)) (justify mirror))
     )
@@
       (effects (font (size 1 1) (thickness 0.15)) (justify mirror))
     )
-    (fp_text value R_Pack04 (at 0 -2.1) (layer B.Fab)
+    (fp_text value 220 (at 0 -2.1) (layer B.Fab)
       (effects (font (size 1 1) (thickness 0.15)) (justify mirror))
     )
@@
       (effects (font (size 1 1) (thickness 0.15)) (justify mirror))
     )
-    (fp_text value R_Pack04 (at 0 -2.1) (layer B.Fab)
-      (effects (font (size 1 1) (thickness 0.15)) (justify mirror))
-    )
+    (fp_text value 220 (at 0 -2.1) (layer B.Fab)
+      (effects (font (size 1 1) (thickness 0.15)) (justify mirror))
+    )
